File: JLCPCB/JLCPCB.kicad_sch (KiCad schematic)
At the start: 1 part

Commit message: #6 Update title blocks
Other:
- title: (none) -> JLCPCB Custom Design Rules (.kicad_dru)
Changed lines of the file:
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@@
 	(generator_version "8.0")
 	(paper "A4")
+	(title_block
+		(title "JLCPCB Custom Design Rules (.kicad_dru)")
+		(date "2024-08-12")
+		(rev "8")
+	)
 	(wire
 		(pts
